File: 2026Car/Main Project/Main Project with Alternator.kicad_sch (KiCad schematic)
At the start: 28 parts, among them K1 Relay_SPST-NO, K2 Relay_SPST-NO, K3 Relay_SPST-NO, SW1 Kill switch, SW2 Brake pull switch, SW3 Reverse switch, SW4 Buzzer button, SW5 Ignition Killswitch, SW6 Load Switch/Signal

Commit message: Final Design Upload
- Separated designs:
1. Main Design - Has no self-charging power source. This is due to a lack of alternator in application, and the magneto can only output a couple of watts (1W being conservative).
2. Main Design w/ Alternator - Main Design + [Alternator -> Filtered Rectifier -> Voltage Regulator -> ±Battery terminals]
General Changelog:
- Added second battery in parallel to main battery due to low Ah rating.
- Diodes have been changed from 1N4148 to a typical Diode (Safety Load measure).
- Design is ready for Reverse Light and a third load, but are placed as DNP due to being unused in the application of said design.
- Changed "Stator" into Magneto; Left Magneto's path as present in real circuit (used to power strictly Car's Ignition).
Parts:
- added C1: 820uF_400V, Capacitor_THT:CP_Radial_D30.0mm_P10.00mm_SnapIn, symbol PCM_SL_Capacitors:470uF_400V
- added C2: 100uF_50V, Capacitor_THT:CP_Radial_D10.0mm_P5.00mm, symbol PCM_SL_Capacitors:470uF_50V
- added D7: W01G, Diode_THT:Diode_Bridge_Round_D9.8mm, symbol Diode_Bridge:W01G
- added F8: Feeding Fuse 20A, symbol Device:Fuse
- added R1: 1k, symbol Device:R_US
- added U1: WG8-40S1203, symbol Converter_DCDC:WG8-40S1203
- added V1: ALT, symbol Simulation_SPICE:VSIN
Connections:
- net GNDPWR: now also D7.2, U1.5 (-Vout), V1.2
- net at BT1.1 (+), BT2.1 (+), F7.1: now also F8.2
- new net: D7.4, V1.1
- new net Input +DC: C1.1, C2.1, D7.1 (+), R1.1, U1.1 (+Vin)
- new net Input -DC: C1.2, C2.2, D7.3 (-), R1.2, U1.2 (-Vin)
- new net Output +DC: F8.1, U1.7 (+Vout)
Other:
- note added: "4B"
- note added: "Circuit ground is designated as the chassis. Alternator is used to charge battery and power the circuit."
- note added: "Power Sources"
- note added: "Stator Rectification and Filtering"
- note added: "Stator Voltage Regulation Input: 8V-40VDC [Min/Max] Output: 13.8VDC @ 20A [Max]"
- note removed: "4A"
- note removed: "Circuit ground is designated as the chassis."
- note removed: "Ignition"
- moved on the sheet: BT1, BT2, BZ1, D1, D2, D3, D4, D5, D6, D8, F1, F2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
